File: light_switch_smd3.brd (EAGLE design)
At the start: 45.7 x 45.7 mm, 26 parts, among them U1 ESP8266_ESP-01

Commit message: added missing sensor data connection
Connections:
- removed net DATA: R11.2, SENSOR.2
- net RXD: now also R11.2, SENSOR.2
Routing:
- net RXD: track 49.4 -> 71.1 mm
- net DATA: track 4.34 -> 0.00 mm
Changed lines of the file:
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@@
 <wire x1="5.588" y1="23.876" x2="12.446" y2="17.018" width="0.3048" layer="16"/>
 <wire x1="12.446" y1="17.018" x2="12.446" y2="5.126" width="0.3048" layer="16"/>
+<contactref element="SENSOR" pad="2"/>
+<contactref element="R11" pad="2"/>
+<wire x1="10.16" y1="27.94" x2="10.16" y2="24.042" width="0.6096" layer="1"/>
+<wire x1="10.16" y1="24.042" x2="9.754" y2="23.876" width="0.762" layer="1"/>
+<wire x1="10.16" y1="27.94" x2="10.16" y2="30.48" width="0.3048" layer="1"/>
+<wire x1="10.16" y1="30.48" x2="7.62" y2="33.02" width="0.3048" layer="1"/>
+<wire x1="7.62" y1="33.02" x2="7.62" y2="40.64" width="0.3048" layer="1"/>
+<wire x1="7.62" y1="40.64" x2="5.362" y2="42.898" width="0.3048" layer="1"/>
+<wire x1="5.362" y1="42.898" x2="4.98" y2="42.898" width="0.3048" layer="1"/>
 </signal>
 <signal name="N$19">
@@
 <wire x1="17.78" y1="25.4" x2="20.32" y2="22.86" width="2.032" layer="16"/>
 </signal>
-<signal name="DATA">
-<contactref element="SENSOR" pad="2"/>
-<contactref element="R11" pad="2"/>
-<wire x1="10.16" y1="27.94" x2="10.16" y2="24.042" width="0.6096" layer="1"/>
-<wire x1="10.16" y1="24.042" x2="9.754" y2="23.876" width="0.762" layer="1"/>
-</signal>
 </signals>
 <mfgpreviewcolors>
@@
 <mfgpreviewcolor name="substratecolor" color="0xFF786E46"/>
 </mfgpreviewcolors>
+<errors>
+</errors>
 </board>
 </drawing>

Commit message: small fixes to be more ERC friendly
Parts:
- SENSOR: value (none) -> CON1
Connections:
- removed net N$13: R1.1
- removed net N$27: R4.1
- removed net N$28: R5.2
- net +3V3: now also R1.1, R4.1, R5.2
Changed lines of the file:
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@@
 <drawing>
 <settings>
-<setting alwaysvectorfont="yes"/>
+<setting alwaysvectorfont="no"/>
 <setting keepoldvectorfont="yes"/>
 <setting verticaltext="up"/>
@@
 <attribute name="NAME" x="18.542" y="18.288" size="0.762" layer="25" font="vector" rot="R270"/>
 </element>
-<element name="SENSOR" library="pinhead" package="1X03" value="" x="10.16" y="27.94" smashed="yes">
+<element name="SENSOR" library="pinhead" package="1X03" value="CON1" x="10.16" y="27.94" smashed="yes">
 <attribute name="NAME" x="9.144" y="29.972" size="0.8128" layer="25" font="vector"/>
-<attribute name="VALUE" x="6.35" y="24.765" size="1.27" layer="27"/>
 </element>
 <element name="R11" library="resistor" package="R1206" value="4.7K" x="11.176" y="23.876" smashed="yes" rot="R180">
@@
 <wire x1="11.278" y1="14.122" x2="14.89755625" y2="14.122" width="0.6096" layer="1"/>
 <wire x1="14.89755625" y1="14.122" x2="15.24" y2="14.46444375" width="0.6096" layer="1"/>
+<contactref element="R1" pad="1"/>
+<contactref element="R4" pad="1"/>
+<contactref element="R5" pad="2"/>
+<wire x1="6.096" y1="10.566" x2="8.636" y2="10.566" width="0" layer="19" extent="16-16"/>
+<wire x1="3.556" y1="10.566" x2="6.096" y2="10.566" width="0" layer="19" extent="16-16"/>
+<wire x1="10.07885" y1="13.72648125" x2="8.636" y2="10.566" width="0" layer="19" extent="1-16"/>
 </signal>
 <signal name="+5V">
@@
 <wire x1="26.1" y1="4.6" x2="25.62" y2="5.08" width="0.6096" layer="1"/>
 <wire x1="25.62" y1="5.08" x2="22.352" y2="5.08" width="0.6096" layer="1"/>
-</signal>
-<signal name="N$28">
-<contactref element="R5" pad="2"/>
 </signal>
 <signal name="GPIO2">
@@
 <wire x1="15.24" y1="43.18" x2="25.4059875" y2="43.18" width="2.032" layer="16"/>
 </signal>
-<signal name="N$13">
-<contactref element="R1" pad="1"/>
-</signal>
-<signal name="N$27">
-<contactref element="R4" pad="1"/>
-</signal>
 <signal name="N$2">

Commit message: routed missed track
Routing:
- net +3V3: track 94.3 -> 112.9 mm, vias 1 -> 2
Changed lines of the file:
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@@
 <contactref element="R4" pad="1"/>
 <contactref element="R5" pad="2"/>
-<wire x1="6.096" y1="10.566" x2="8.636" y2="10.566" width="0" layer="19" extent="16-16"/>
-<wire x1="3.556" y1="10.566" x2="6.096" y2="10.566" width="0" layer="19" extent="16-16"/>
-<wire x1="10.07885" y1="13.72648125" x2="8.636" y2="10.566" width="0" layer="19" extent="1-16"/>
+<wire x1="3.556" y1="10.566" x2="6.096" y2="10.566" width="0.3048" layer="16"/>
+<wire x1="6.096" y1="10.566" x2="8.636" y2="10.566" width="0.3048" layer="16"/>
+<wire x1="8.636" y1="10.566" x2="8.636" y2="16.764" width="0.3048" layer="16"/>
+<wire x1="8.636" y1="16.764" x2="7.62" y2="17.78" width="0.3048" layer="16"/>
+<via x="7.62" y="17.78" extent="1-16" drill="0.35"/>
+<wire x1="7.62" y1="17.78" x2="10.464" y2="17.78" width="0.6096" layer="1"/>
+<wire x1="10.464" y1="17.78" x2="12.598" y2="19.914" width="0.6096" layer="1"/>
 </signal>
 <signal name="+5V">
